Commit message: mape_loop issue with LiDAR subscription

File: install/robot_description/share/robot_description/urdf/robot.xacro (robot description, xacro)
@@ -2,7 +2,12 @@
 <robot name="robot" xmlns:xacro="http://www.ros.org/wiki/xacro">
     <xacro:include filename="$(find robot_description)/urdf/robot.gazebo" />
+    <xacro:include filename="$(find robot_description)/urdf/marker.xacro" />
     <!-- Link - base_link -->
     <link name="base_link"></link>
-    <!-- Joint - base_link/chassis -->
+    <!-- place marker on robot-->
+    <xacro:marker prefix="marker12" parent="link_chassis">
+        <origin xyz="0 0 0.07" rpy= "0 0 0"/>
+    </xacro:marker>
+<!-- Joint - base_link/chassis -->
     <joint name="joint_base_link_chassis" type="fixed">
         <origin rpy="0 0 0" xyz="0 0 0" />
