Commit message: experiments with different distance parameter

File: install/robot_description/share/robot_description/urdf/marker.xacro (robot description, xacro)
@@ -6,5 +6,5 @@
     <link name="${prefix}_link">
       <visual>
-        <origin xyz="0 0 0" rpy="0 1.57 0"/>
+        <origin xyz="0 0 0" rpy="0 -1.57 0"/>
         <xacro:insert_block name="origin"/>
         <geometry>

Commit message: v7 does not use orientation

File: install/robot_description/share/robot_description/urdf/marker.xacro (robot description, xacro)
@@ -6,8 +6,8 @@
     <link name="${prefix}_link">
       <visual>
-        <origin xyz="0 0 0" rpy="0 -1.57 0"/>
+        <origin xyz="0 0 0" rpy="0 1.57 0"/>
         <xacro:insert_block name="origin"/>
         <geometry>
-          <mesh filename="model://marker12/meshes/Marker12.dae" scale ="0.2 0.2 0.2"/>
+          <mesh filename="model://marker12/meshes/Marker12.dae" scale ="0.3 0.3 0.3"/>
         </geometry>
       </visual>
